Commit message: failed localization by amcl

File: nhk2021_simulator/urdf/lidar.urdf.xacro (robot description, xacro)
@@ -26,5 +26,5 @@
         <pose>0 0 0 0 0 0</pose>
         <visualize>false</visualize>
-        <update_rate>10</update_rate>
+        <update_rate>20</update_rate>
         <ray>
           <scan>
@@ -44,5 +44,5 @@
             <type>gaussian</type>
             <mean>0.0</mean>
-            <stddev>0.0</stddev>
+            <stddev>0.01</stddev>
           </noise>
         </ray>

File: nhk2021_simulator/urdf/wheel.urdf.xacro (robot description, xacro)
@@ -3,5 +3,5 @@
 <xacro:property name="PI" value="3.1415926535897931"/>
 <xacro:property name="wheel_radius" value="0.035"/>
-<xacro:property name="wheel_height" value="0.05"/>
+<xacro:property name="wheel_height" value="0.06"/>
 <xacro:property name="wheel_mass" value="0.50"/>
 <xacro:macro name="wheel" params="rl parent">
@@ -31,8 +31,8 @@
   <child link="wheel_${rl}" />
   <xacro:if value="${rl == 'r'}">
-    <origin xyz="0 -0.22 0.035" rpy="${PI/2} 0 0" /><!--z: position from base_link - position from body-->
+    <origin xyz="0 -0.25 0.035" rpy="${PI/2} 0 0" /><!--z: position from base_link - position from body-->
   </xacro:if>
   <xacro:if value="${rl == 'l'}">
-     <origin xyz="0 0.22 0.035" rpy="${PI/2} 0 0" />
+     <origin xyz="0 0.25 0.035" rpy="${PI/2} 0 0" />
   </xacro:if>
   <axis xyz="0 0 -1" />
