Commit message: FEAT: add BBox

File: nhk2021_simulator/urdf/_d435.gazebo.xacro (robot description, xacro)
@@ -25,5 +25,5 @@
       <sensor name="${camera_name}color" type="camera">
         <camera name="${camera_name}">
-          <horizontal_fov>${69.4*deg_to_rad}</horizontal_fov>
+          <horizontal_fov>${85.2*deg_to_rad}</horizontal_fov>
           <image>
           <!--
@@ -95,5 +95,5 @@
       <sensor name="${camera_name}depth" type="depth">
         <camera name="${camera_name}">
-          <horizontal_fov>${69.4*deg_to_rad}</horizontal_fov><!--85.2-->
+          <horizontal_fov>${85.2*deg_to_rad}</horizontal_fov><!--85.2-->
           <image>
             <width>1280</width>

File: nhk2021_simulator/urdf/swerve_robot.urdf.xacro (robot description, xacro)
@@ -20,5 +20,5 @@
  <xacro:imu_macro prefix="imu" parent="base_footprint" xyz="0.0 0 0.10" />
  <sensor_d435 parent="rplidar_link">
-    <origin xyz="0.0 0.0 0.3" rpy="0 0 0"/>
+    <origin xyz="0.0 0.0 1.0" rpy="0 0.1745 0"/>
   </sensor_d435>
 </robot>
