Commit message: add realsense model

File: nhk2021_simulator/urdf/swerve_robot.urdf.xacro (robot description, xacro)
@@ -5,4 +5,5 @@
  <xacro:include filename="$(find nhk2021_simulator)/urdf/lidar.urdf.xacro" />
  <xacro:include filename="$(find nhk2021_simulator)/urdf/imu.urdf.xacro" />
+ <xacro:include filename="$(find nhk2021_simulator)/urdf/_d435.urdf.xacro" />
   <gazebo>
     <plugin name="gazebo_ros_control" filename="libgazebo_ros_control.so">
@@ -18,3 +19,6 @@
  <xacro:laser_macro prefix="rplidar" parent="base_footprint" xyz="0.205 0 0.04" />
  <xacro:imu_macro prefix="imu" parent="base_footprint" xyz="0.0 0 0.10" />
+ <sensor_d435 parent="rplidar_link">
+    <origin xyz="0.0 0.0 0.3" rpy="0 0 0"/>
+  </sensor_d435>
 </robot>

Commit message: FEAT: add path

File: nhk2021_simulator/urdf/swerve_robot.urdf.xacro (robot description, xacro)
@@ -20,5 +20,5 @@
  <xacro:imu_macro prefix="imu" parent="base_footprint" xyz="0.0 0 0.10" />
  <sensor_d435 parent="rplidar_link">
-    <origin xyz="0.0 0.0 1.0" rpy="0 0.1745 0"/>
+    <origin xyz="0.0 0.0 0.3" rpy="0 0.1745 0"/>
   </sensor_d435>
 </robot>
