Commit message: FEAR: initial_table_angle

File: nhk2021_simulator/urdf/swerve_wheel.urdf.xacro (robot description, xacro)
@@ -54,5 +54,5 @@
   <parent link="wheel_${rl}_round_table" />
   <child link="wheel_${rl}" />
-  <origin xyz="0.0 -0.05 0.0" rpy="0 0 0" /><!--z: position from base_link - position from body-->
+  <origin xyz="0.0 -0.05 0.0" rpy="0 ${PI/2} 0" /><!--z: position from base_link - position from body-->
   <axis xyz="0 0 -1" />
   <limit effort="6.0" velocity="60.0" /><!-- maximum torqe(<8.82), maximum velocity-->
